File: pcb/pcb.kicad_pcb (KiCad board)
At the start: 2 copper layers, 347.7 x 133.4 mm, 254 parts, among them J1 USB_C_Receptacle_USB2.0_16P, SW1 SW_Push, U1 SRV05-4_C7420376, U2 XC6206P332MR, U3 STM32F072CBTx

Commit message: jlcpcb USB-C
Parts:
- J1: value USB_C_Receptacle_USB2.0_16P -> Connector, USB-TYPE-C-16P; footprint PCM_marbastlib-various:USB_C_Receptacle_HRO_TYPE-C-31-M-12 -> PCM_JLCPCB:TYPE-C-SMD_HX-TYPE-C-16PIN
- moved J1 1.49 mm to (335.0, 33.5)
- moved R2 0.40 mm to (337.5, 37.5)
- moved R1 0.37 mm to (332.6, 37.5)
Routing:
- net GND: track 26.4 -> 25.6 mm
